File: EMC Assignment 2.kicad_pcb (KiCad board)
At the start: 2 copper layers, 90 parts, among them IC1 LP2985AIM5-3.0_NOPB, J1 M40-3200445R, U1 LT8636, U2 ATMEGA16U2-MU, U3 ATMEGA328P-PU, U4 OPA4350, U5 OPA4350, U6 OPA4350, U7 OPA4350, X2 USB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

Commit message: Some layout around U1 has been done
Parts:
- moved U2 77.9 mm to (36.0, 83.0)
- moved AD1 67.9 mm to (116.6, 83.6)
- moved BLM21 67.9 mm to (145.4, 93.0)
- moved C25 67.9 mm to (162.9, 102.6)
- moved C26 67.9 mm to (162.9, 105.6)
- moved C4 67.9 mm to (92.0, 93.2)
- moved L2 67.9 mm to (138.6, 87.1)
- moved R10 67.9 mm to (162.8, 114.6)
- moved R11 67.9 mm to (162.8, 117.5)
- moved R3 67.9 mm to (158.4, 114.6)
- moved R4 67.9 mm to (158.4, 117.5)
- moved U3 67.9 mm to (83.8, 109.3)
- moved W1 67.9 mm to (136.7, 94.8)
- moved C1 67.9 mm to (158.4, 99.6)
- moved C11 67.9 mm to (95.9, 127.2)
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
Commit message: U1 layout sketch done
Parts:
- moved C16 24.8 mm to (39.5, 33.5), turned to -90 degrees
- moved R6 23.5 mm to (36.5, 28.5)
- moved R8 17.6 mm to (36.5, 26.0)
- moved C19 11.2 mm to (39.5, 38.4), turned to -90 degrees
- moved L3 3.54 mm to (39.5, 42.5)
- moved C18 0.67 mm to (35.0, 39.0)
Changed lines of the file:
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@@
 		(tags "Integrated Circuit")
 		(property "Reference" "U1"
-			(at 1 -4 0)
+			(at 5 -3.5 0)
 			(layer "F.SilkS")
 			(effects
@@
 	(footprint "Resistor_SMD:R_0805_2012Metric"
 		(layer "F.Cu")
-		(at 60 29)
+		(at 36.5 28.5)
 		(descr "Resistor SMD 0805 (2012 Metric), square (rectangular) end terminal, IPC_7351 nominal, (Body size source: IPC-SM-782 page 72, https://www.pcb-3d.com/wordpress/wp-content/uploads/ipc-sm-782a_amendment_1_and_2.pdf), generated with kicad-footprint-generator")
 		(tags "resistor")
 		(property "Reference" "R6"
-			(at 0 -1.65 0)
+			(at 3 0 0)
 			(layer "F.SilkS")
 			(effects
@@
 	(footprint "C0805C112F5GACTU//:C0805"
 		(layer "F.Cu")
-		(at 60.6 46.5)
+		(at 39.5 33.5 -90)
 		(descr "C0805")
 		(tags "Capacitor")
 		(property "Reference" "C16"
-			(at 0 0 0)
+			(at 0 0 90)
 			(layer "F.SilkS")
 			(effects
@@
 		)
 		(property "Value" "1uF"
-			(at 0 0 0)
+			(at 0 0 90)
 			(layer "F.SilkS")
 			(hide yes)
@@
 		)
 		(property "Footprint" "C0805C112F5GACTU//:C0805"
-			(at 0 0 0)
+			(at 0 0 -90)
 			(unlocked yes)
 			(layer "F.Fab")
@@
 		)
 		(property "Datasheet" ""
-			(at 0 0 0)
+			(at 0 0 -90)
 			(unlocked yes)
 			(layer "F.Fab")
@@
 		)
 		(property "Description" "Unpolarized capacitor"
-			(at 0 0 0)
+			(at 0 0 -90)
 			(unlocked yes)
 			(layer "F.Fab")
@@
 		)
 		(fp_line
-			(start -2.275 -1.625)
-			(end 2.275 -1.625)
+			(start -2.275 1.625)
+			(end -2.275 -1.625)
 			(stroke
 				(width 0.05)
@@
 		)
 		(fp_line
-			(start -2.275 1.625)
-			(end -2.275 -1.625)
+			(start 2.275 1.625)
+			(end -2.275 1.625)
 			(stroke
 				(width 0.05)
@@
 		)
 		(fp_line
-			(start 2.275 -1.625)
-			(end 2.275 1.625)
+			(start -2.275 -1.625)
+			(end 2.275 -1.625)
 			(stroke
 				(width 0.05)
@@
 		)
 		(fp_line
-			(start 2.275 1.625)
-			(end -2.275 1.625)
+			(start 2.275 -1.625)
+			(end 2.275 1.625)
 			(stroke
 				(width 0.05)
@@
 		)
 		(fp_line
-			(start -1 -0.625)
-			(end 1 -0.625)
+			(start -1 0.625)
+			(end -1 -0.625)
 			(stroke
 				(width 0.2)
@@
 		)
 		(fp_line
-			(start -1 0.625)
-			(end -1 -0.625)
+			(start 1 0.625)
+			(end -1 0.625)
 			(stroke
 				(width 0.2)
@@
 		)
 		(fp_line
-			(start 1 -0.625)
-			(end 1 0.625)
+			(start -1 -0.625)
+			(end 1 -0.625)
 			(stroke
 				(width 0.2)
@@
 		)
 		(fp_line
-			(start 1 0.625)
-			(end -1 0.625)
+			(start 1 -0.625)
+			(end 1 0.625)
 			(stroke
 				(width 0.2)
@@
 		)
 		(fp_text user "${REFERENCE}"
-			(at 0 0 0)
+			(at 0 0 90)
 			(layer "F.Fab")
 			(effects
@@
 		)
 		(pad "1" smd rect
-			(at -0.9 0)
+			(at -0.9 0 270)
 			(size 1.15 1.45)
 			(layers "F.Cu" "F.Paste" "F.Mask")
@@
 		)
 		(pad "2" smd rect
-			(at 0.9 0)
+			(at 0.9 0 270)
 			(size 1.15 1.45)
 			(layers "F.Cu" "F.Paste" "F.Mask")
@@
 	(footprint "C0805C112F5GACTU//:C0805"
 		(layer "F.Cu")
-		(at 34.7 39.6 180)
+		(at 35 39 180)
 		(descr "C0805")
 		(tags "Capacitor")
 		(property "Reference" "C18"
-			(at -3.9 0 360)
+			(at 0.2 -2.4 360)
 			(layer "F.SilkS")
 			(effects
@@
 	(footprint "Inductor_SMD:L_0805_2012Metric"
 		(layer "F.Cu")
-		(at 37 45 90)
+		(at 39.5 42.5 90)
 		(descr "Inductor SMD 0805 (2012 Metric), square (rectangular) end terminal, IPC_7351 nominal, (Body size source: IPC-SM-782 page 80, https://www.pcb-3d.com/wordpress/wp-content/uploads/ipc-sm-782a_amendment_1_and_2.pdf), generated with kicad-footprint-generator")
 		(tags "inductor")
@@
 	(footprint "C0805C112F5GACTU//:C0805"
 		(layer "F.Cu")
-		(at 44.4 48.5)
+		(at 39.5 38.4 -90)
 		(descr "C0805")
 		(tags "Capacitor")
 		(property "Reference" "C19"
-			(at 0 0 0)
+			(at 0 0 90)
 			(layer "F.SilkS")
 			(effects
@@
 		)
 		(property "Value" "1uF"
-			(at 0 0 0)
+			(at 0 0 90)
 			(layer "F.SilkS")
 			(hide yes)
@@
 		)
 		(property "Footprint" "C0805C112F5GACTU//:C0805"
-			(at 0 0 0)
+			(at 0 0 -90)
 			(unlocked yes)
 			(layer "F.Fab")
@@
 		)
 		(property "Datasheet" ""
-			(at 0 0 0)
+			(at 0 0 -90)
 			(unlocked yes)
 			(layer "F.Fab")
@@
 		)
 		(property "Description" "Unpolarized capacitor"
-			(at 0 0 0)
+			(at 0 0 -90)
 			(unlocked yes)
 			(layer "F.Fab")
@@
 		)
 		(fp_line
-			(start -2.275 -1.625)
-			(end 2.275 -1.625)
+			(start -2.275 1.625)
+			(end -2.275 -1.625)
 			(stroke
 				(width 0.05)
@@
 		)
 		(fp_line
-			(start -2.275 1.625)
-			(end -2.275 -1.625)
+			(start 2.275 1.625)
+			(end -2.275 1.625)
 			(stroke
 				(width 0.05)
@@
 		)
 		(fp_line
-			(start 2.275 -1.625)
-			(end 2.275 1.625)
+			(start -2.275 -1.625)
+			(end 2.275 -1.625)
 			(stroke
 				(width 0.05)
@@
 		)
 		(fp_line
-			(start 2.275 1.625)
-			(end -2.275 1.625)
+			(start 2.275 -1.625)
+			(end 2.275 1.625)
 			(stroke
 				(width 0.05)
@@
 		)
 		(fp_line
-			(start -1 -0.625)
-			(end 1 -0.625)
+			(start -1 0.625)
+			(end -1 -0.625)
 			(stroke
 				(width 0.2)
@@
 		)
 		(fp_line
-			(start -1 0.625)
-			(end -1 -0.625)
+			(start 1 0.625)
+			(end -1 0.625)
 			(stroke
 				(width 0.2)
@@
 		)
 		(fp_line
-			(start 1 -0.625)
-			(end 1 0.625)
+			(start -1 -0.625)
+			(end 1 -0.625)
 			(stroke
 				(width 0.2)
@@
 		)
 		(fp_line
-			(start 1 0.625)
-			(end -1 0.625)
+			(start 1 -0.625)
+			(end 1 0.625)
 			(stroke
 				(width 0.2)
@@
 		)
 		(fp_text user "${REFERENCE}"
-			(at 0 0 0)
+			(at 0 0 90)
 			(layer "F.Fab")
 			(effects
@@
 		)
 		(pad "1" smd rect
-			(at -0.9 0)
+			(at -0.9 0 270)
 			(size 1.15 1.45)
 			(layers "F.Cu" "F.Paste" "F.Mask")
@@
 		)
 		(pad "2" smd rect
-			(at 0.9 0)
+			(at 0.9 0 270)
 			(size 1.15 1.45)
 			(layers "F.Cu" "F.Paste" "F.Mask")
@@
 	(footprint "Resistor_SMD:R_0805_2012Metric"
 		(layer "F.Cu")
-		(at 48.9125 38.5)
+		(at 36.5 26)
 		(descr "Resistor SMD 0805 (2012 Metric), square (rectangular) end terminal, IPC_7351 nominal, (Body size source: IPC-SM-782 page 72, https://www.pcb-3d.com/wordpress/wp-content/uploads/ipc-sm-782a_amendment_1_and_2.pdf), generated with kicad-footprint-generator")
 		(tags "resistor")
 		(property "Reference" "R8"
-			(at 0 -1.65 0)
+			(at 3 0 360)
 			(layer "F.SilkS")
 			(effects
@@
 		)
 		(property "Value" "243k"
-			(at 0 1.65 0)
+			(at 0 1.65 360)
 			(layer "F.Fab")
 			(effects
@@
 		)
 		(fp_text user "${REFERENCE}"
-			(at 0 0 0)
+			(at 0 0 360)
 			(layer "F.Fab")
 			(effects

Commit message: More stuff done
Parts:
- removed C29: 100nF, Capacitor_SMD:C_0805_2012Metric
- removed C30, C31, C32, C33: 30pF, Capacitor_SMD:C_0805_2012Metric
- removed RR1: 47, Resistor_SMD:R_0805_2012Metric
- removed U4, U5, U6, U7: OPA4350, Package_SO:SOIC-8_3.9x4.9mm_P1.27mm
- added C24: 30pF, Capacitor_SMD:C_0805_2012Metric, F.Cu at (90.5, 63.0)
- added C34: 100nF, Capacitor_SMD:C_0805_2012Metric, F.Cu at (84.5, 73.5)
- added C35: 10nF, Capacitor_SMD:C_0805_2012Metric, F.Cu at (90.5, 69.0)
- added C37: 30pF, Capacitor_SMD:C_0805_2012Metric, F.Cu at (90.5, 52.5)
- added C5: 10nF, Capacitor_SMD:C_0805_2012Metric, F.Cu at (111.5, 62.0)
- added R18: 10k, Resistor_SMD:R_0805_2012Metric, F.Cu at (90.5, 66.5)
- added U8: OPA4350EA_250, emc:OPA4350 SOP64P600X175-16N, F.Cu at (98.0, 57.5)
- AD1: footprint 87891-0808:HDRV8W69P0X254_1X8_2032X251X1641P -> emc:HDRV8W69P0X254_1X8_2032X251X1641P
- C10, C11, C11B1, C12, C13, C14, C15, C16, C17, C18, C19, C20, C4, C6, C7, C8, C9, C9B1: footprint C0805C112F5GACTU//:C0805 -> emc:C0805
- C25: value 10nF -> 30pF
- C26: value 100nF -> 30pF
- C27: value 100nF -> 10nF
- F1: footprint MF-MSMF050-2:FUSC4632X85N -> emc:FUSC4632X85N
- IC1: footprint LIB_LP2985AIM5-3.0_NOPB(1):SOT95P280X145-5N -> emc:SOT95P280X145-5N
- ICSP1, ICSP2: footprint M22-5320305R:M225320305R -> emc:M225320305R
- IO1: footprint B10B-XASK-1(LF)(SN):SHDR10W64P0X250_1X10_2740X575X700P -> emc:SHDR10W64P0X250_1X10_2740X575X700P
- J1: footprint M40-3200445R:HUSSP8W30P100_2X4_400X320X365P -> emc:HUSSP8W30P100_2X4_400X320X365P
- JP2: footprint M20-7820446:RHDR4W70P0X254_1X4_1056X250X865P -> emc:RHDR4W70P0X254_1X4_1056X250X865P
- R13: value 10k -> 47
- U1: footprint LT8636HV#PBF:LT8636HVPBF -> emc:LT8636HVPBF
- U2: footprint ATMEGA16U2-MU:QFN50P500X500X100-33N-D -> emc:QFN50P500X500X100-33N-D
- U3: footprint ATMEGA328P-PU//:DIP794W53P254L3467H457Q28N -> emc:DIP794W53P254L3467H457Q28N
- moved R11 121.9 mm to (96.9, 15.0)
- moved RN4A1 118.7 mm to (27.5, 48.6), turned to -90 degrees
- moved R4 116.1 mm to (104.0, 15.0), turned to 180 degrees
- moved IO1 116.1 mm to (14.5, 46.5), turned to -90 degrees
- moved R3 115.2 mm to (100.5, 15.0), turned to 180 degrees
- moved JP2 114.6 mm to (88.0, 14.0), turned to 180 degrees
- moved R5 114.2 mm to (106.0, 19.0), turned to 90 degrees
- moved RN3B1 113.9 mm to (67.0, 21.5), turned to 90 degrees
- moved RN3A1 112.2 mm to (65.0, 21.5), turned to 90 degrees
- moved RN4B1 111.4 mm to (29.5, 48.6), turned to -90 degrees
- moved C11 106.9 mm to (58.6, 27.0)
- moved ICSP1 106.6 mm to (54.0, 38.5)
- moved Z1 102.6 mm to (64.5, 17.5)
- moved Z2 102.3 mm to (68.0, 17.5), turned to 180 degrees
- moved BLM21 100.7 mm to (73.5, 22.4), turned to 90 degrees
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Connections:
- C2 pad 1: Net-(C2-Pad1) -> Net-(U8-+IN_B)
- C2 pad 2: Net-(U4--) -> GND
- C21 pad 1: Net-(C21-Pad1) -> Net-(U8-+IN_C)
- C21 pad 2: Net-(U7--) -> GND
- C22 pad 1: Net-(U4-+) -> Net-(C22-Pad1)
- C22 pad 2: GND -> Net-(U8--IN_D)
- C23 pad 1: Net-(U5-+) -> Net-(U8-+IN_D)
- C25 pad 1: Net-(U7-+) -> /AD2
- C25 pad 2: GND -> Net-(U8--V)
- C26 pad 1: +3.3V -> /AD3
- C26 pad 2: GND -> Net-(U8--V)
- C27 pad 1: +3.3V -> Net-(U8-+IN_A)
- R10 pad 1: Net-(C2-Pad1) -> Net-(C5-Pad1)
- R10 pad 2: Net-(U4-+) -> Net-(U8-+IN_C)
- R11 pad 1: Net-(C3-Pad1) -> Net-(C22-Pad1)
- R11 pad 2: Net-(U5-+) -> /ADCD
- R12 pad 1: Net-(C5-Pad1) -> Net-(C22-Pad1)
- R12 pad 2: Net-(U6-+) -> Net-(U8-+IN_D)
- R13 pad 1: Net-(C21-Pad1) -> /AD1
- R13 pad 2: Net-(U7-+) -> Net-(U8-OUT_B)
- R14 pad 1: Net-(R14-Pad1) -> /AD2
- R14 pad 2: /AD0 -> Net-(U8-OUT_C)
- R15 pad 1: Net-(R15-Pad1) -> /AD3
- R15 pad 2: /AD1 -> Net-(U8-OUT_D)
- R16 pad 1: Net-(R16-Pad1) -> /AD0
- R16 pad 2: /AD3 -> Net-(U8-OUT_A)
- R3 pad 1: Net-(C2-Pad1) -> Net-(C3-Pad1)
- R3 pad 2: /ADCA -> /ADCB
- R4 pad 1: Net-(C3-Pad1) -> Net-(U8-+IN_B)
- R4 pad 2: /ADCA -> Net-(C3-Pad1)
- R5 pad 1: Net-(C5-Pad1) -> Net-(C35-Pad2)
- R9 pad 1: Net-(C21-Pad1) -> Net-(C5-Pad1)
- R9 pad 2: /ADCA -> /ADCC
