File: EMC Assignment 2.kicad_sch (KiCad schematic)
At the start: 88 parts, among them IC1 LP2985AIM5-3.0_NOPB, J1 M40-3200445R, U1 LT8636, U2 ATMEGA16U2-MU, U3 ATMEGA328P-PU, U8 OPA4350EA_250, X2 USB, Y1 16MHz, Y2 16M

Commit message: 3/4 of blocks done
Parts:
- BLM21: footprint BLM21:BLM21AG102BH1J -> emc:BLM21AG102BH1J
- C10, C11B1, C4, C6, C9B1: footprint C0805C112F5GACTU//:C0805 -> emc:C0805
- C11, C12, C13, C14, C15, C16, C17, C18, C19, C20, C7, C8, C9: footprint C0805C112F5GACTU//:C0805 -> Capacitor_SMD:C_0805_2012Metric
- POWER1: footprint 3-647166-2// -> emc:36471662
- Z1, Z2: footprint CG0603MLC-05E:VARC1608X55N -> emc:VARC1608X55N
Connections:
- net GND: now also C16.2, C19.1, C24.2, C25.2, C26.2, C37.2, R6.2, R8.2, U1.13 (GND_2), U1.21 (GND_3), U8.13 (-V)
Changed lines of the file:
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@@
 	)
 	(junction
+		(at 119.38 46.99)
+		(diameter 0)
+		(color 0 0 0 0)
+	)
+	(junction
 		(at 30.48 242.57)
 		(diameter 0)
@@
 	)
 	(junction
+		(at 342.9 110.49)
+		(diameter 0)
+		(color 0 0 0 0)
+	)
+	(junction
 		(at 45.72 49.53)
 		(diameter 0)
@@
 	(wire
 		(pts
+			(xy 119.38 46.99) (xy 119.38 41.91)
+		)
+		(stroke
+			(width 0)
+			(type default)
+		)
+	)
+	(wire
+		(pts
 			(xy 48.26 215.9) (xy 54.61 215.9)
 		)
@@
 	(wire
 		(pts
+			(xy 119.38 46.99) (xy 127 46.99)
+		)
+		(stroke
+			(width 0)
+			(type default)
+		)
+	)
+	(wire
+		(pts
 			(xy 303.53 120.65) (xy 326.39 120.65)
 		)
@@
 	(wire
 		(pts
-			(xy 328.93 110.49) (xy 364.49 110.49)
+			(xy 328.93 110.49) (xy 342.9 110.49)
 		)
 		(stroke
@@
 	(wire
 		(pts
+			(xy 342.9 110.49) (xy 342.9 115.57)
+		)
+		(stroke
+			(width 0)
+			(type default)
+		)
+	)
+	(wire
+		(pts
 			(xy 215.9 118.11) (xy 199.39 118.11)
 		)
@@
 	(wire
 		(pts
+			(xy 342.9 110.49) (xy 364.49 110.49)
+		)
+		(stroke
+			(width 0)
+			(type default)
+		)
+	)
+	(wire
+		(pts
 			(xy 322.58 77.47) (xy 328.93 77.47)
 		)
@@
 	(wire
 		(pts
-			(xy 119.38 49.53) (xy 119.38 41.91)
+			(xy 119.38 49.53) (xy 119.38 46.99)
 		)
 		(stroke
@@
 			)
 		)
-		(property "Footprint" "C0805C112F5GACTU//:C0805"
+		(property "Footprint" "Capacitor_SMD:C_0805_2012Metric"
 			(at 49.2252 41.91 0)
 			(effects
@@
 			)
 		)
-		(property "Footprint" "C0805C112F5GACTU//:C0805"
+		(property "Footprint" "Capacitor_SMD:C_0805_2012Metric"
 			(at 177.8 129.8448 0)
 			(effects
@@
 			)
 		)
-		(property "Footprint" "C0805C112F5GACTU//:C0805"
+		(property "Footprint" "Capacitor_SMD:C_0805_2012Metric"
 			(at 46.6852 49.53 0)
 			(effects
@@
 			)
 		)
-		(property "Footprint" "C0805C112F5GACTU//:C0805"
+		(property "Footprint" "emc:C0805"
 			(at 26.67 245.4148 0)
 			(effects
@@
 			)
 		)
-		(property "Footprint" "C0805C112F5GACTU//:C0805"
+		(property "Footprint" "Capacitor_SMD:C_0805_2012Metric"
 			(at 45.72 106.9848 0)
 			(effects
@@
 			)
 		)
-		(property "Footprint" "C0805C112F5GACTU//:C0805"
+		(property "Footprint" "emc:C0805"
 			(at 140.6652 259.08 0)
 			(effects
@@
 			)
 		)
-		(property "Footprint" "CG0603MLC-05E:VARC1608X55N"
+		(property "Footprint" "emc:VARC1608X55N"
 			(at 200.914 134.874 90)
 			(effects
@@
 			)
 		)
-		(property "Footprint" "BLM21:BLM21AG102BH1J"
+		(property "Footprint" "emc:BLM21AG102BH1J"
 			(at 187.96 130.81 0)
 			(effects
@@
 			)
 		)
-		(property "Footprint" "C0805C112F5GACTU//:C0805"
+		(property "Footprint" "Capacitor_SMD:C_0805_2012Metric"
 			(at 45.72 114.6048 0)
 			(effects
@@
 			)
 		)
-		(property "Footprint" "C0805C112F5GACTU//:C0805"
+		(property "Footprint" "Capacitor_SMD:C_0805_2012Metric"
 			(at 33.9852 49.53 0)
 			(effects
@@
 			)
 		)
-		(property "Footprint" "C0805C112F5GACTU//:C0805"
+		(property "Footprint" "Capacitor_SMD:C_0805_2012Metric"
 			(at 58.42 56.1848 0)
 			(effects
@@
 			)
 		)
-		(property "Footprint" "C0805C112F5GACTU//:C0805"
+		(property "Footprint" "emc:C0805"
 			(at 25.4 260.6548 0)
 			(effects
@@
 			)
 		)
-		(property "Footprint" "CG0603MLC-05E:VARC1608X55N"
+		(property "Footprint" "emc:VARC1608X55N"
 			(at 200.914 138.684 90)
 			(effects
@@
 			)
 		)
-		(property "Footprint" "C0805C112F5GACTU//:C0805"
+		(property "Footprint" "Capacitor_SMD:C_0805_2012Metric"
 			(at 45.72 98.0948 0)
 			(effects
@@
 			)
 		)
-		(property "Footprint" "C0805C112F5GACTU//:C0805"
+		(property "Footprint" "emc:C0805"
 			(at 201.93 255.5748 0)
 			(effects
@@
 			)
 		)
-		(property "Footprint" "3-647166-2//"
+		(property "Footprint" "emc:36471662"
 			(at 34.29 163.5 0)
 			(effects
@@
 			)
 		)
-		(property "Footprint" "C0805C112F5GACTU//:C0805"
+		(property "Footprint" "Capacitor_SMD:C_0805_2012Metric"
 			(at 120.3452 64.77 0)
 			(effects
@@
 			)
 		)
-		(property "Footprint" "C0805C112F5GACTU//:C0805"
+		(property "Footprint" "Capacitor_SMD:C_0805_2012Metric"
 			(at 67.31 48.5648 0)
 			(effects
@@
 			)
 		)
-		(property "Footprint" "C0805C112F5GACTU//:C0805"
+		(property "Footprint" "emc:C0805"
 			(at 31.4452 242.57 0)
 			(effects
@@
 			)
 		)
-		(property "Footprint" "C0805C112F5GACTU//:C0805"
+		(property "Footprint" "Capacitor_SMD:C_0805_2012Metric"
 			(at 58.1152 30.48 0)
 			(effects
@@
 	(symbol
 		(lib_id "power:GND")
+		(at 342.9 115.57 0)
+		(unit 1)
+		(exclude_from_sim no)
+		(in_bom yes)
+		(on_board yes)
+		(dnp no)
+		(fields_autoplaced yes)
+		(property "Reference" "#PWR030"
+			(at 342.9 121.92 0)
+			(effects
+				(font
+					(size 1.27 1.27)
+				)
+				(hide yes)
+			)
+		)
+		(property "Value" "GND"
+			(at 342.9 120.65 0)
+			(effects
+				(font
+					(size 1.27 1.27)
+				)
+			)
+		)
+		(property "Footprint" ""
+			(at 342.9 115.57 0)
+			(effects
+				(font
+					(size 1.27 1.27)
+				)
+				(hide yes)
+			)
+		)
+		(property "Datasheet" ""
+			(at 342.9 115.57 0)
+			(effects
+				(font
+					(size 1.27 1.27)
+				)
+				(hide yes)
+			)
+		)
+		(property "Description" ""
+			(at 342.9 115.57 0)
+			(effects
+				(font
+					(size 1.27 1.27)
+				)
+				(hide yes)
+			)
+		)
+		(pin "1"
+		)
+		(instances
+			(project "EMC Assignment 2"
+				(path "/73140039-e75b-4089-b60b-1534d1c3d425"
+					(reference "#PWR030")
+					(unit 1)
+				)
+			)
+		)
+	)
+	(symbol
+		(lib_id "power:GND")
 		(at 299.72 76.2 0)
 		(unit 1)
@@
 			)
 		)
-		(property "Footprint" "C0805C112F5GACTU//:C0805"
+		(property "Footprint" "Capacitor_SMD:C_0805_2012Metric"
 			(at 118.11 48.5648 0)
 			(effects
@@
 	)
 	(symbol
+		(lib_id "power:GND")
+		(at 127 46.99 0)
+		(unit 1)
+		(exclude_from_sim no)
+		(in_bom yes)
+		(on_board yes)
+		(dnp no)
+		(fields_autoplaced yes)
+		(property "Reference" "#PWR031"
+			(at 127 53.34 0)
+			(effects
+				(font
+					(size 1.27 1.27)
+				)
+				(hide yes)
+			)
+		)
+		(property "Value" "GND"
+			(at 127 52.07 0)
+			(effects
+				(font
+					(size 1.27 1.27)
+				)
+			)
+		)
+		(property "Footprint" ""
+			(at 127 46.99 0)
+			(effects
+				(font
+					(size 1.27 1.27)
+				)
+				(hide yes)
+			)
+		)
+		(property "Datasheet" ""
+			(at 127 46.99 0)
+			(effects
+				(font
+					(size 1.27 1.27)
+				)
+				(hide yes)
+			)
+		)
+		(property "Description" "Power symbol creates a global label with name \"GND\" , ground"
+			(at 127 46.99 0)
+			(effects
+				(font
+					(size 1.27 1.27)
+				)
+				(hide yes)
+			)
+		)
+		(pin "1"
+		)
+		(instances
+			(project "EMC Assignment 2"
+				(path "/73140039-e75b-4089-b60b-1534d1c3d425"
+					(reference "#PWR031")
+					(unit 1)
+				)
+			)
+		)
+	)
+	(symbol
 		(lib_id "Device:R_US")
 		(at 39.37 254 0)
@@
 			)
 		)
-		(property "Footprint" "C0805C112F5GACTU//:C0805"
+		(property "Footprint" "Capacitor_SMD:C_0805_2012Metric"
 			(at 22.5552 49.53 0)
 			(effects
