File: EMC Assignment 2.kicad_sch (KiCad schematic)
At the start: 88 parts, among them IC1 LP2985AIM5-3.0_NOPB, J1 M40-3200445R, U1 LT8636, U2 ATMEGA16U2-MU, U3 ATMEGA328P-PU, U8 OPA4350EA_250, X2 USB, Y1 16MHz, Y2 16M

Commit message: pcb done
Parts:
- C10, C11B1, C4, C6, C9B1: footprint emc:C0805 -> Capacitor_SMD:C_0805_2012Metric
Connections:
- net GND: now also BLM21.2, X2.5 (GND)
Changed lines of the file:
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@@
 	)
 	(junction
+		(at 220.98 130.81)
+		(diameter 0)
+		(color 0 0 0 0)
+	)
+	(junction
 		(at 30.48 242.57)
 		(diameter 0)
@@
 	(wire
 		(pts
+			(xy 220.98 130.81) (xy 220.98 134.62)
+		)
+		(stroke
+			(width 0)
+			(type default)
+		)
+	)
+	(wire
+		(pts
 			(xy 24.13 156.21) (xy 29.21 156.21)
 		)
@@
 			)
 		)
-		(property "Footprint" "emc:C0805"
+		(property "Footprint" "Capacitor_SMD:C_0805_2012Metric"
 			(at 26.67 245.4148 0)
 			(effects
@@
 			)
 		)
-		(property "Footprint" "emc:C0805"
+		(property "Footprint" "Capacitor_SMD:C_0805_2012Metric"
 			(at 140.6652 259.08 0)
 			(effects
@@
 	)
 	(symbol
+		(lib_id "power:GND")
+		(at 220.98 134.62 0)
+		(unit 1)
+		(exclude_from_sim no)
+		(in_bom yes)
+		(on_board yes)
+		(dnp no)
+		(fields_autoplaced yes)
+		(property "Reference" "#PWR032"
+			(at 220.98 140.97 0)
+			(effects
+				(font
+					(size 1.27 1.27)
+				)
+				(hide yes)
+			)
+		)
+		(property "Value" "GND"
+			(at 220.98 139.7 0)
+			(effects
+				(font
+					(size 1.27 1.27)
+				)
+			)
+		)
+		(property "Footprint" ""
+			(at 220.98 134.62 0)
+			(effects
+				(font
+					(size 1.27 1.27)
+				)
+				(hide yes)
+			)
+		)
+		(property "Datasheet" ""
+			(at 220.98 134.62 0)
+			(effects
+				(font
+					(size 1.27 1.27)
+				)
+				(hide yes)
+			)
+		)
+		(property "Description" "Power symbol creates a global label with name \"GND\" , ground"
+			(at 220.98 134.62 0)
+			(effects
+				(font
+					(size 1.27 1.27)
+				)
+				(hide yes)
+			)
+		)
+		(pin "1"
+		)
+		(instances
+			(project "EMC Assignment 2"
+				(path "/73140039-e75b-4089-b60b-1534d1c3d425"
+					(reference "#PWR032")
+					(unit 1)
+				)
+			)
+		)
+	)
+	(symbol
 		(lib_id "Device:C")
 		(at 21.59 261.62 90)
@@
 			)
 		)
-		(property "Footprint" "emc:C0805"
+		(property "Footprint" "Capacitor_SMD:C_0805_2012Metric"
 			(at 25.4 260.6548 0)
 			(effects
@@
 			)
 		)
-		(property "Footprint" "emc:C0805"
+		(property "Footprint" "Capacitor_SMD:C_0805_2012Metric"
 			(at 201.93 255.5748 0)
 			(effects
@@
 			)
 		)
-		(property "Footprint" "emc:C0805"
+		(property "Footprint" "Capacitor_SMD:C_0805_2012Metric"
 			(at 31.4452 242.57 0)
 			(effects
